File: Slothboard_V2.kicad_pcb (KiCad board)
At the start: 2 copper layers, 101 x 32 mm, 43 parts, among them J1 1x3_pinHeader, J2 1x3_pinHeader, J3 1x3_pinHeader, J4 1x3_pinHeader, J5 1x4_PinHeader, J6 1x4_PinHeader, J7 1x4_PinHeader, Q1 AO3401A, SW1 SW_MEC_5E, U1 CYTLP185, U2 STM32F303RBTx, U3 AMS1117-3.3, U4 1x2_pinheader

Commit message: added more photos
Changed lines of the file:
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@@
     (property "Sheetfile" "Slothboard_V2.kicad_sch")
     (property "Sheetname" "")
-    (attr through_hole)
+    (attr through_hole exclude_from_bom)
     (fp_text reference "J6" (at 4.385 -2.27 90) (layer "F.SilkS")
       (effects (font (size 1 1) (thickness 0.15)))
@@
     (property "Sheetfile" "Slothboard_V2.kicad_sch")
     (property "Sheetname" "")
-    (attr through_hole)
+    (attr through_hole exclude_from_bom)
     (fp_text reference "J5" (at 4.385 -2.27 90) (layer "F.SilkS")
       (effects (font (size 1 1) (thickness 0.15)))
@@
     (property "Sheetfile" "Slothboard_V2.kicad_sch")
     (property "Sheetname" "")
-    (attr exclude_from_pos_files)
+    (attr exclude_from_pos_files exclude_from_bom)
     (fp_text reference "H1" (at -0.01 3.22) (layer "F.SilkS")
       (effects (font (size 1 1) (thickness 0.15)))
@@
     )
   )
-  (footprint "Logos:ES_LOGO" (layer "F.Cu")
+  (footprint "Logos:ES_LOGO" locked (layer "F.Cu")
     (at 192.4 51.8)
-    (attr board_only exclude_from_pos_files exclude_from_bom)
+    (attr board_only exclude_from_pos_files)
     (fp_text reference "G***" (at -2.81 -3.25) (layer "F.Fab")
       (effects (font (size 1.524 1.524) (thickness 0.3)))
@@
     (property "Sheetfile" "Slothboard_V2.kicad_sch")
     (property "Sheetname" "")
-    (attr through_hole)
+    (attr through_hole exclude_from_bom)
     (fp_text reference "U4" (at -3.05 -0.115 180) (layer "F.SilkS")
       (effects (font (size 1 1) (thickness 0.15)))
@@
     (property "Sheetfile" "Slothboard_V2.kicad_sch")
     (property "Sheetname" "")
-    (attr exclude_from_pos_files)
+    (attr exclude_from_pos_files exclude_from_bom)
     (fp_text reference "H3" (at 0 -3.2) (layer "F.SilkS")
       (effects (font (size 1 1) (thickness 0.15)))
@@
     (property "Sheetfile" "Slothboard_V2.kicad_sch")
     (property "Sheetname" "")
-    (attr exclude_from_pos_files)
+    (attr exclude_from_pos_files exclude_from_bom)
     (fp_text reference "H2" (at 0 -3.2) (layer "F.SilkS")
       (effects (font (size 1 1) (thickness 0.15)))
@@
     (property "Sheetname" "")
     (attr smd)
-    (fp_text reference "D1" (at 0.6 -1.8 90 unlocked) (layer "F.SilkS")
+    (fp_text reference "D1" (at 0.0638 -1.6542 90 unlocked) (layer "F.SilkS")
       (effects (font (size 1 1) (thickness 0.15)))
     )
@@
     (property "Sheetfile" "Slothboard_V2.kicad_sch")
     (property "Sheetname" "")
-    (attr exclude_from_pos_files)
+    (attr exclude_from_pos_files exclude_from_bom)
     (fp_text reference "H4" (at 0 3.5) (layer "F.SilkS")
       (effects (font (size 1 1) (thickness 0.15)))
@@
   (via (at 117.85 68.32) (size 0.8) (drill 0.4) (layers "F.Cu" "B.Cu") (free) (net 2))
   (via (at 162.116809 54.616809) (size 0.8) (drill 0.4) (layers "F.Cu" "B.Cu") (net 2))
-  (via (at 128.5 72) (size 0.8) (drill 0.4) (layers "F.Cu" "B.Cu") (free) (net 2))
+  (via (at 128.88 72.02) (size 0.8) (drill 0.4) (layers "F.Cu" "B.Cu") (free) (net 2))
   (via (at 155.14 57.8) (size 0.8) (drill 0.4) (layers "F.Cu" "B.Cu") (net 2))
   (via (at 149.2 64.4) (size 0.8) (drill 0.4) (layers "F.Cu" "B.Cu") (net 2))
   (via (at 141.96 67.21) (size 0.8) (drill 0.4) (layers "F.Cu" "B.Cu") (free) (net 2))
-  (via (at 132.35 66.8) (size 0.8) (drill 0.4) (layers "F.Cu" "B.Cu") (free) (net 2))
+  (via (at 132.39 66.89) (size 0.8) (drill 0.4) (layers "F.Cu" "B.Cu") (free) (net 2))
   (via (at 179.44 67.82) (size 0.8) (drill 0.4) (layers "F.Cu" "B.Cu") (net 2))
   (via (at 156 70.5) (size 0.8) (drill 0.4) (layers "F.Cu" "B.Cu") (free) (net 2))
@@
   (via (at 186.175 68.25) (size 0.8) (drill 0.4) (layers "F.Cu" "B.Cu") (net 2))
   (via (at 184.975 68.225) (size 0.8) (drill 0.4) (layers "F.Cu" "B.Cu") (net 2))
-  (via (at 109.5 69) (size 0.8) (drill 0.4) (layers "F.Cu" "B.Cu") (free) (net 2))
+  (via (at 110.03 68.98) (size 0.8) (drill 0.4) (layers "F.Cu" "B.Cu") (free) (net 2))
   (via (at 154.75 76.71) (size 0.8) (drill 0.4) (layers "F.Cu" "B.Cu") (net 2))
   (via (at 145.25 49.17) (size 0.8) (drill 0.4) (layers "F.Cu" "B.Cu") (net 2))
