File: Slothboard_V2.kicad_sch (KiCad schematic)
At the start: 42 parts, among them J1 1x3_pinHeader, J2 1x3_pinHeader, J3 1x3_pinHeader, J4 1x3_pinHeader, J5 1x4_PinHeader, J6 1x4_PinHeader, J7 1x4_PinHeader, Q1 AO3401A, SW1 SW_MEC_5E, U1 CYTLP185, U2 STM32F303RBTx, U3 AMS1117-3.3, U4 1x2_pinheader

Commit message: added more photos
Parts:
- C1: JLCPCB Part # (none) -> C19666
- C10, C2, C3, C4, C5, C6: JLCPCB Part # (none) -> C14663
- C11, C12: JLCPCB Part # (none) -> C129303
- C7: JLCPCB Part # (none) -> C57112
- C8, C9: JLCPCB Part # (none) -> C15849
- D1, D2, D4: value G_LED -> Y_LED; JLCPCB Part # (none) -> C2296
- D3: JLCPCB Part # (none) -> C84256
- FB1: value 600@100MHz -> 100@100MHz; JLCPCB Part # (none) -> C1015
- Q1: JLCPCB Part # (none) -> C15127
- R1, R2, R6, R7, R8: JLCPCB Part # (none) -> C17513
- R3: JLCPCB Part # (none) -> C17414
- R4, R5: JLCPCB Part # (none) -> C17520
- U1: JLCPCB Part # (none) -> C385052
- U2: JLCPCB Part # (none) -> C130453; LCSC Part # (none) -> C130453
- U3: JLCPCB Part # (none) -> C6186
Other:
- note added: "12v maximun because of the max VGS of the AO3401A (12v max) NOTE: An Zenner diode can be added to clamp the VGS voltage"
- note removed: "12v maximun because of the max VGS of the AO3401A (12v max) NOTE: An Zenner diode can be added to limit the VGS voltage"
